File: Kicad/Desktop_weather_station/Desktop_weather_station.sch (KiCad schematic (older format))
At the start: 3 parts, among them U1 TCRT5000

Commit message: update
Parts:
- removed U1: TCRT5000, TCRT5000:OPTO_TCRT5000, symbol TCRT5000:TCRT5000
- added C1: 10mk, Capacitor_Tantalum_SMD:CP_EIA-3216-18_Kemet-A, symbol Device:C
- added C2, C3, C6: 0.1, Capacitor_SMD:C_0603_1608Metric_Pad1.08x0.95mm_HandSolder, symbol Device:C
- added C4, C5: 22p, Capacitor_SMD:C_0603_1608Metric_Pad1.08x0.95mm_HandSolder, symbol Device:C
- added D1: SS14, Diode_SMD:D_SMA, symbol Device:D
- added D2: 1N4001, Diode_SMD:D_SMA, symbol Device:D
- added F1: 100mA, Fuse:Fuse_1206_3216Metric_Pad1.42x1.75mm_HandSolder, symbol Device:Polyfuse
- added J1: Batt 3V7, symbol Connector_Generic:Conn_01x02
- added J2: Antenna, symbol Connector_Generic:Conn_01x02
- added J3: LCD, Connector_PinHeader_2.54mm:PinHeader_1x08_P2.54mm_Vertical, symbol Connector_Generic:Conn_01x08
- added J4: UART, symbol Connector_Generic:Conn_01x03
- added R3: 100R, Resistor_SMD:R_0805_2012Metric_Pad1.20x1.40mm_HandSolder, symbol Device:R
- added SW1: SW_MEC_5G, symbol Switch:SW_MEC_5G
- added U1: DS18B20, Package_TO_SOT_THT:TO-92_Inline, symbol Sensor_Temperature:DS18B20
- added U2: ATmega328P-AU, Package_QFP:TQFP-32_7x7mm_P0.8mm, symbol MCU_Microchip_ATmega:ATmega328P-AU
- added U3: CC1101_E07, symbol CC1101:CC1101_E07
- added Y1: 8MHz, Crystal:Crystal_HC49-4H_Vertical, symbol Device:Crystal
- R1: value 470R -> 4k7
- R2: value 100k -> 10k
Connections:
- net GND: now also C1.2, C2.2, C3.2, C4.1, C5.2, C6.2, J1.2 (Pin_2), J2.2 (Pin_2), J3.2 (Pin_2), J4.3 (Pin_3), SW1.1 (A), SW1.2 (A), U1.1 (GND), U2.21 (GND), U2.3 (GND), U2.5 (GND), U3.10 (GND), U3.8 (GND)
- net AD0: now reaches R1.2
- net AD0: now also U1.2 (DQ), U2.23 (PC0)
- net +5V: no longer names the net of R2.1
- net +5V: now also C1.1, C3.1, D1.1 (K), D2.2 (A), J3.1 (Pin_1), U2.18 (AVCC), U2.4 (VCC), U2.6 (VCC)
- net proximity_sensor_led renamed D7
- net D7: now also U1.3 (VDD), U2.11 (PD7)
- net proximity_sensor_to_mcu renamed RESET
- net RESET: now also U2.29 (~RESET~/PC6)
- new net: C2.1, U2.20 (AREF)
- new net: C4.2, U2.7 (XTAL1/PB6), Y1.1
- new net: C5.1, U2.8 (XTAL2/PB7), Y1.2
- new net: C6.1, D2.1 (K), U3.1 (VCC)
- new net: J2.1 (Pin_1), U3.9 (ANT)
- new net: D1.2 (A), F1.1
- new net: J3.8 (Pin_8), R3.1
- new net +BATT: F1.2, J1.1 (Pin_1)
- new net AD1: U2.24 (PC1)
- new net AD2: U2.25 (PC2)
- new net AD3: U2.26 (PC3)
- new net AD4: U2.27 (PC4)
- new net AD5: U2.28 (PC5)
- new net D0: J4.1 (Pin_1), U2.30 (PD0)
- new net D1: J4.2 (Pin_2), U2.31 (PD1)
- new net D10: U2.14 (PB2), U3.3 (CSN)
- new net D11: J3.6 (Pin_6), U2.15 (PB3), U3.5 (MOSI)
- new net D12: U2.16 (PB4), U3.6 (MISO/GDO1)
- new net D13: J3.7 (Pin_7), U2.17 (PB5), U3.4 (SCK)
- new net D2: U2.32 (PD2), U3.7 (GDO2)
- new net D3: SW1.3 (B), SW1.4 (B), U2.1 (PD3)
- new net D4: J3.3 (Pin_3), U2.2 (PD4)
- new net D5: R3.2, U2.9 (PD5)
- new net D6: U2.10 (PD6), U3.2 (GDO0)
- new net D8: J3.5 (Pin_5), U2.12 (PB0)
- new net D9: J3.4 (Pin_4), U2.13 (PB1)
- no-connect marks 0 -> 2
Other:
- note added: "ILI9163 1.44"
- note added: "a0"
- note added: "cs"
- note added: "gnd"
- note added: "led"
- note added: "reset"
- note added: "sck"
- note added: "sda"
- note added: "vcc"
